Commit message: things

File: urdf/car.urdf.xacro (robot description, xacro)
@@ -9,6 +9,6 @@
     <link name="base_link">
         <visual>
-            <geometry><box size="0.6 0.4 0.2"/></geometry>
-            <origin xyz="0 0 0.1" rpy="0 0 0"/>
+            <geometry><box size="0.42 0.25 0.15"/></geometry>
+            <origin xyz="0 0 0.0725" rpy="0 0 0"/>
             <material name="green"/>
         </visual>
@@ -17,5 +17,5 @@
         <visual>
             <geometry>
-                <cylinder radius="0.1" length="0.05"/>
+                <cylinder radius="0.05" length="0.04"/>
             </geometry>
             <origin xyz="0 0 0" rpy="1.57 0 0"/>
@@ -26,5 +26,5 @@
         <visual>
             <geometry>
-                <cylinder radius="0.1" length="0.05"/>
+                <cylinder radius="0.05" length="0.04"/>
             </geometry>
             <origin xyz="0 0 0" rpy="1.57 0 0"/>
@@ -35,5 +35,5 @@
         <visual>
             <geometry>
-                <cylinder radius="0.1" length="0.05"/>
+                <cylinder radius="0.05" length="0.04"/>
             </geometry>
             <origin xyz="0 0 0" rpy="1.57 0 0"/>
@@ -44,5 +44,5 @@
         <visual>
             <geometry>
-                <cylinder radius="0.1" length="0.05"/>
+                <cylinder radius="0.05" length="0.04"/>
             </geometry>
             <origin xyz="0 0 0" rpy="1.57 0 0"/>
@@ -53,5 +53,5 @@
         <parent link="base_link" />
         <child link="front_left_wheel" />
-        <origin xyz="0.15 0.255 0" rpy="0 0 0" />
+        <origin xyz="0.16 0.125 0" rpy="0 0 0" />
         <axis xyz="0 1 0" />
     </joint>
@@ -59,5 +59,5 @@
         <parent link="base_link" />
         <child link="front_right_wheel" />
-        <origin xyz="0.15 -0.255 0" rpy="0 0 0" />
+        <origin xyz="0.16 -0.125 0" rpy="0 0 0" />
         <axis xyz="0 1 0" />
     </joint>
@@ -65,5 +65,5 @@
         <parent link="base_link" />
         <child link="back_left_wheel" />
-        <origin xyz="-0.15 0.255 0" rpy="0 0 0" />
+        <origin xyz="-0.16 0.125 0" rpy="0 0 0" />
         <axis xyz="0 1 0" />
     </joint>
@@ -71,5 +71,5 @@
         <parent link="base_link" />
         <child link="back_right_wheel" />
-        <origin xyz="-0.15 -0.255 0" rpy="0 0 0" />
+        <origin xyz="-0.16 -0.125 0" rpy="0 0 0" />
         <axis xyz="0 1 0" />
     </joint>

File: urdf/robot_integration.urdf.xacro (robot description, xacro)
@@ -34,5 +34,5 @@
       <parent link="zed_camera_link"/>
       <child link="base_link"/>
-      <origin xyz="-0.3 0.0 -0.20" rpy="0 0 0"/>
+      <origin xyz="-0.21 0.0 -0.17" rpy="0 0 0"/>
     </joint>
   </xacro:if>
@@ -41,5 +41,5 @@
       <parent link="base_link"/>
       <child link="zed_camera_link"/>
-      <origin xyz="0.3 0.0 0.20" rpy="0 0 0"/>
+      <origin xyz="0.21 0.0 0.15" rpy="0 0 0"/>
     </joint>
   </xacro:unless>
@@ -48,6 +48,6 @@
 <joint name="vesc_joint" type="fixed">
   <parent link="base_link"/>
-  <child link="vesc_base_link"/>
-  <origin xyz="-0.0 0 0.20" rpy="0 0 0"/>
+  <child link="vesc/base_link"/>
+  <origin xyz="-0.0 -0.03 0.13" rpy="0 0 0"/>
 </joint>
 </robot>

File: urdf/vesc.urdf.xacro (robot description, xacro)
@@ -4,5 +4,5 @@
   <xacro:macro name="vesc" params="name:=vesc">
     <!-- VESC Base Link -->
-    <link name="${name}_base_link">
+    <link name="vesc/base_link">
       <visual>
         <origin xyz="0 0 0" rpy="0 0 0"/>
